File: CSI1802X.sch (KiCad schematic (older format))
At the start: 4 parts

Commit message: smoothing caps
Parts:
- added C?: 0.1uF, ~, symbol C_CER
- added C?: 3300uF, ~, symbol C_EL
- D? (x4): value DIODE -> 1N5402
Connections:
- wire segments 12 -> 16
Changed lines of the file:
@@
 P 3250 3050
 F 0 "D?" H 3250 3150 40  0000 C CNN
-F 1 "DIODE" H 3250 2950 40  0000 C CNN
+F 1 "1N5402" H 3250 2950 40  0000 C CNN
 F 2 "~" H 3250 3050 60  0000 C CNN
 F 3 "~" H 3250 3050 60  0000 C CNN
@@
 P 2850 3700
 F 0 "D?" H 2850 3800 40  0000 C CNN
-F 1 "DIODE" H 2850 3600 40  0000 C CNN
+F 1 "1N5402" H 2850 3600 40  0000 C CNN
 F 2 "~" H 2850 3700 60  0000 C CNN
 F 3 "~" H 2850 3700 60  0000 C CNN
@@
 P 3650 3700
 F 0 "D?" H 3650 3800 40  0000 C CNN
-F 1 "DIODE" H 3650 3600 40  0000 C CNN
+F 1 "1N5402" H 3650 3600 40  0000 C CNN
 F 2 "~" H 3650 3700 60  0000 C CNN
 F 3 "~" H 3650 3700 60  0000 C CNN
@@
 P 3250 4000
 F 0 "D?" H 3250 4100 40  0000 C CNN
-F 1 "DIODE" H 3250 3900 40  0000 C CNN
+F 1 "1N5402" H 3250 3900 40  0000 C CNN
 F 2 "~" H 3250 4000 60  0000 C CNN
 F 3 "~" H 3250 4000 60  0000 C CNN
@@
 $EndComp
 Wire Wire Line
-	2450 4000 3050 4000
+	2150 4000 3050 4000
 Wire Wire Line
 	3450 4000 4100 4000
@@
 Connection ~ 2850 4000
 Wire Wire Line
-	2500 3050 3050 3050
+	2150 3050 3050 3050
 Wire Wire Line
 	3450 3050 4050 3050
@@
 	2950 3150 2950 3050
 Connection ~ 2950 3050
+$Comp
+L C_CER C?
+U 1 1 533A0E65
+P 2450 3600
+F 0 "C?" H 2470 3660 30  0000 L BNN
+F 1 "0.1uF" H 2470 3540 30  0000 L TNN
+F 2 "~" H 2488 3450 30  0000 C CNN
+F 3 "~" H 2450 3600 60  0000 C CNN
+	1    2450 3600
+	1    0    0    -1
+$EndComp
+Wire Wire Line
+	2450 3800 2450 4000
+Connection ~ 2450 4000
+Wire Wire Line
+	2450 3400 2450 3050
+Connection ~ 2450 3050
+$Comp
+L C_EL C?
+U 1 1 533A0EEF
+P 4000 3550
+F 0 "C?" H 4020 3610 30  0000 L BNN
+F 1 "3300uF" H 4020 3460 30  0000 L TNN
+F 2 "~" H 4038 3400 30  0000 C CNN
+F 3 "~" H 4000 3550 60  0000 C CNN
+	1    4000 3550
+	1    0    0    -1
+$EndComp
+Wire Wire Line
+	4000 3350 4000 3050
+Connection ~ 4000 3050
+Wire Wire Line
+	4000 3750 4000 4000
+Connection ~ 4000 4000
 $EndSCHEMATC
